File: Schema/hardware/Projet_schematics.sch (KiCad schematic (older format))
At the start: 21 parts, among them J1 Prog Header, U1 PIC16LF1789, U2 UA78M33CDCY, U3 LMT87LP, U4 OPT101P, U5 HIH-5030-001, U6 410-340, U7 MICS-VZ-89TE, U8 RN42-I/RM630

Commit message: Update shematics
Parts:
- removed C5: 33pF, symbol Device:C
- removed R2, R3: 4.7kΩ, symbol Device:R
- removed U4: OPT101P, symbol Project:OPT101P
- removed U6: 410-340, symbol Project:410-340
- removed U7: MICS-VZ-89TE, symbol Project:MICS-VZ-89TE
- added D2: LED, symbol Device:LED
- added R1: PDV-P8001, symbol Device:R_PHOTO
- added R5: 220Ω, symbol Device:R
- C1: value 0.33µF -> 100µF
- C3: value 0.1µF -> 10µF
- R2: renamed from R1; value 100kΩ -> 4.7kΩ
- renumbered R5 to R3, U5 to U4, U8 to U5
Connections:
- wire segments 156 -> 100
Other:
- moved on the sheet: R2, U5
